File: PCB_Design_GSM_GPS/GSM_GPS/GSM_GPS.kicad_sch (KiCad schematic)
At the start: 25 parts, among them J1 SIM8051-6-0-14-00-X-REVD, J2 Conn_01x03_Pin, J3 Conn_01x03_Pin, J4 Conn_01x03_Pin, J5 Conn_01x03_Pin, J6 Conn_01x03_Pin, Q1 2N3904, U1 SIM868

Commit message: Update full schematic
Parts:
- removed D1: D_Zener, symbol Device:D_Zener
- removed J4: Conn_01x03_Pin, symbol Connector:Conn_01x03_Pin
- added AE1: GGBLA.01.A, GGBLA.01.A:XCVR_GGBLA.01.A, symbol GGBLA.01.A:GGBLA.01.A
- added C10, C19: 0.1uF, Capacitor_SMD:C_0201_0603Metric, symbol Device:C_Small
- added C11, C14: 0.5pF, Capacitor_SMD:C_0201_0603Metric, symbol Device:C_Small
- added C12: 1uF, Capacitor_SMD:C_0201_0603Metric, symbol Device:C_Small
- added C13: 0.8pF, Capacitor_SMD:C_0201_0603Metric, symbol Device:C_Small
- added C15: 22pF, Capacitor_SMD:C_0201_0603Metric, symbol Device:C_Small
- added C16: 100uF, Capacitor_SMD:CP_Elec_6.3x7.7, symbol Device:C_Polarized
- added C18: 330uF, Capacitor_SMD:CP_Elec_8x10.5, symbol Device:C_Polarized
- added C23: 2.7pF, Capacitor_SMD:C_0201_0603Metric, symbol Device:C_Small
- added C7, C8, C9: 22pF, Capacitor_SMD:C_0402_1005Metric, symbol Device:C_Small
- added D4: ESDA6V1-5SC6, Package_TO_SOT_SMD:SOT-23-6, symbol Power_Protection:ESDA6V1-5SC6
- added D5: 5.1V, Diode_SMD:D_0201_0603Metric, symbol Device:D_Zener
- added E1: YC0003AA, YC0003AA:XCVR_YC0003AA, symbol YC0003AA:YC0003AA
- added J10, J11, J8, J9: Conn_01x03_Pin, Connector_Molex:Molex_SPOX_5267-03A_1x03_P2.50mm_Vertical, symbol Connector:Conn_01x03_Pin
- added J12, J13, J14, J15, J16, J17, J18, J19, J4: Conn_01x04_Pin, Connector_Molex:Molex_SPOX_5267-04A_1x04_P2.50mm_Vertical, symbol Connector:Conn_01x04_Pin
- added J20, J21, J7: Conn_01x02_Pin, Connector_Molex:Molex_SPOX_5267-02A_1x02_P2.50mm_Vertical, symbol Connector:Conn_01x02_Pin
- added L1: 3.3nH, Inductor_SMD:L_0402_1005Metric, symbol Device:L
- added L2: 6.8nH, Inductor_SMD:L_0201_0603Metric, symbol Device:L
- added R10: 43k, Resistor_SMD:R_0805_2012Metric, symbol Device:R
- added R11: 470k, Resistor_SMD:R_0201_0603Metric, symbol Device:R
- added R9: 10k, Resistor_SMD:R_0201_0603Metric, symbol Device:R
- added U2: SeeeduinoXIAO nRF52840 Sense, Seeed Studio XIAO Series Library:XIAO-nRF52840-Sense-14P-2.54-21X17.8MM, symbol Seeeduino XIAO:SeeeduinoXIAO
- added U3: MIC29302AWD, Package_TO_SOT_SMD:TO-252-5_TabPin3, symbol Regulator_Linear:MIC29302AWD
- C1, C4: footprint (none) -> Capacitor_SMD:C_0805_2012Metric
- C2, C3: footprint (none) -> Capacitor_SMD:C_1210_3225Metric
- C5: footprint (none) -> Capacitor_SMD:C_0201_0603Metric
- C6: footprint (none) -> Capacitor_SMD:C_0402_1005Metric
- J2, J3, J5, J6: footprint (none) -> Connector_Molex:Molex_SPOX_5267-03A_1x03_P2.50mm_Vertical
- R1, R2, R3, R5, R6, R7, R8: footprint (none) -> Resistor_SMD:R_0201_0603Metric
- R4: value 22 -> 100k; footprint (none) -> Resistor_SMD:R_0201_0603Metric
Connections:
- net UART2_RX is gone; now on net GPS_RX: U1.23 (UART2_RXD)
- net UART2_TX is gone; now on net GPS_TX: U1.22 (UART2_TXD)
- net GND: now also AE1.2 (gnd), C10.2, C11.2, C12.2, C13.2, C15.2, C16.2, C18.2, C19.2, C7.2, C8.2, C9.2, D4.2 (GND), D5.2 (A), J10.3 (Pin_3), J11.3 (Pin_3), J12.4 (Pin_4), J13.4 (Pin_4), J14.4 (Pin_4), J16.1 (Pin_1), J16.2 (Pin_2), J16.3 (Pin_3), J16.4 (Pin_4), J20.2 (Pin_2), J21.2 (Pin_2), J4.4 (Pin_4), J7.2 (Pin_2), J8.3 (Pin_3), J9.3 (Pin_3), L2.2, R10.2, R11.2, U2.13 (GND), U3.3 (GND)
- net GPS_EN: now also R9.2
- net GPS_RX: now also J4.1 (Pin_1)
- net GPS_TX: now also J4.2 (Pin_2)
- net VCC: no longer C1.1, C2.1, C3.1, C4.1, C5.1, C6.1, U1.28 (VRTC), U1.34 (GPS_VBAT), U1.35 (VBAT)
- net at R4.2: now also R10.1, U3.5 (ADJ); no longer U1.14 (SIM1_DET)
- net at J1.C1 (VCC), U1.18 (SIM1_VDD): now also C10.1, D4.3 (IO2)
- net GSM_ANT: now reaches U1.32 (GSM_ANT)
- net GSM_ANT: now also L1.2
- net POWER_PIN: now reaches Q1.3 (C), U1.39 (PWRKEY)
- net POWER_PIN: now also J7.1 (Pin_1)
- net GPIO1: now reaches U1.57 (GPIO1)
- net GPIO1: now also J15.2 (Pin_2), J4.3 (Pin_3), U2.2 (PA4_A1_D1)
- net GPS_ANT: now reaches U1.68 (GPS_ANT)
- net GPS_ANT: now also C23.2
- net at J1.C3 (CLK), R2.1: now also C8.1, D4.5 (IO4)
- net at J1.C6 (VPP): no longer R4.1
- net at J1.C7 (I/O), R1.1: now also C9.1, D4.4 (IO3)
- net at J1.C2 (RST), R3.1: now also C7.1, D4.6 (IO5)
- new net: AE1.1 (RF_Feed), C13.1, C14.2, C23.1
- new net: C11.1, E1.1, L1.1
- new net: E1.2, L2.1
- new net: AE1.3 (FTE), C14.1, C15.1
- new net BATTERY_IN: C12.1, C16.1, J20.1 (Pin_1), U3.1 (EN), U3.2 (VIN)
- new net GPIO0: J15.1 (Pin_1), U2.1 (PA02_A0_D0)
- new net GPIO2: J15.3 (Pin_3), U2.3 (PA10_A2_D2)
- new net GPIO3: J15.4 (Pin_4), U2.4 (PA11_A3_D3)
- new net GPS_EN_GPIO1: J21.1 (Pin_1), R9.1
- new net SIM868_Vin: C1.1, C18.1, C19.1, C2.1, C3.1, C4.1, C5.1, C6.1, D5.1 (K), J19.1 (Pin_1), J19.2 (Pin_2), J19.3 (Pin_3), J19.4 (Pin_4), R11.1, R4.1, U1.28 (VRTC), U1.34 (GPS_VBAT), U1.35 (VBAT), U3.4 (VOUT)
- new net XIAO_3.3V: J17.1 (Pin_1), J17.2 (Pin_2), J17.3 (Pin_3), J17.4 (Pin_4), U2.12 (3V3)
- new net XIAO_5V: J18.1 (Pin_1), J18.2 (Pin_2), J18.3 (Pin_3), J18.4 (Pin_4), U2.14 (5V)
- new net XIAO_I2C_SCL: J10.2 (Pin_2), J11.2 (Pin_2), J9.2 (Pin_2), U2.6 (PA9_A5_D5_SCL)
- new net XIAO_I2C_SDA: J10.1 (Pin_1), J11.1 (Pin_1), J9.1 (Pin_1), U2.5 (PA8_A4_D4_SDA)
- new net XIAO_SPI_MISO: J12.2 (Pin_2), J13.2 (Pin_2), J14.2 (Pin_2), U2.10 (PA5_A9_D9_MISO)
- new net XIAO_SPI_MOSI: J12.1 (Pin_1), J13.1 (Pin_1), J14.1 (Pin_1), U2.11 (PA6_A10_D10_MOSI)
- new net XIAO_SPI_SCK: J12.3 (Pin_3), J13.3 (Pin_3), J14.3 (Pin_3), U2.9 (PA7_A8_D8_SCK)
- new net XIAO_UART_RX: J8.2 (Pin_2), U2.8 (PB09_A7_D7_RX)
- new net XIAO_UART_TX: J8.1 (Pin_1), U2.7 (PB08_A6_D6_TX)
Other:
- note added: "13 November 2023"
- note added: "GSM_VBAT: Min: 3.4V, Max: 4.4V GPS_VBAT: Min: 2.9V, Max: 4.4V VRTC : Min: 2.3V, Max: 4.3V"
- note added: "SEOW SIN KIAT"
- note added: "Seeed XIAO nRF52840 Sense & SIM868"
- moved on the sheet: C1, C2, C3, C4, C5, C6, D2, D3, J1, J2, J3, J5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

Commit message: Update new schematic
Parts:
- removed AE1: GGBLA.01.A, GGBLA.01.A:XCVR_GGBLA.01.A, symbol GGBLA.01.A:GGBLA.01.A
- removed C13: 0.8pF, Capacitor_SMD:C_0201_0603Metric, symbol Device:C_Small
- removed C14: 0.5pF, Capacitor_SMD:C_0201_0603Metric, symbol Device:C_Small
- removed C15: 22pF, Capacitor_SMD:C_0201_0603Metric, symbol Device:C_Small
- removed C16: 100uF, Capacitor_SMD:CP_Elec_6.3x7.7, symbol Device:C_Polarized
- removed C18: 330uF, Capacitor_SMD:CP_Elec_8x10.5, symbol Device:C_Polarized
- removed C2, C3: 330uF, Capacitor_SMD:C_1210_3225Metric, symbol Device:C_Small
- removed C23: 2.7pF, Capacitor_SMD:C_0201_0603Metric, symbol Device:C_Small
- added C12: 100uF, Capacitor_SMD:CP_Elec_6.3x5.4, symbol Device:C_Polarized_Small
- added C14, C2, C3: 330uF, Capacitor_SMD:CP_Elec_8x10.5, symbol Device:C_Polarized_Small
- added E2: ACAG0301-1575-T, ACAG0301-1575-T:ANT_ACAG0301-1575-T, symbol ACAG0301-1575-T:ACAG0301-1575-T
- added L3: 2.4nH, Inductor_SMD:L_0201_0603Metric, symbol Device:L
- added L4: 5.6nH, Inductor_SMD:L_0201_0603Metric, symbol Device:L
- D2, D3: footprint LED_SMD:LED_0201_0603Metric_Pad0.64x0.40mm_HandSolder -> LED_SMD:LED_0201_0603Metric
- D5: value 5.1V -> 5.1V/500mW
- L2: footprint Inductor_SMD:L_0201_0603Metric -> Inductor_SMD:L_01005_0402Metric
- R1, R2, R3: footprint Resistor_SMD:R_0201_0603Metric -> Resistor_SMD:R_0603_1608Metric
- R10: footprint Resistor_SMD:R_0805_2012Metric -> Resistor_SMD:R_1210_3225Metric
- R11: footprint Resistor_SMD:R_0201_0603Metric -> Resistor_SMD:R_1210_3225Metric
- R4: renamed from R5; footprint Resistor_SMD:R_0201_0603Metric -> Resistor_SMD:R_0805_2012Metric
- R5: renamed from R6; footprint Resistor_SMD:R_0201_0603Metric -> Resistor_SMD:R_0805_2012Metric
- R6: renamed from R7; value 4.7k -> 40; footprint Resistor_SMD:R_0201_0603Metric -> Resistor_SMD:R_1206_3216Metric
- R7: renamed from R8; value 4.7k -> 40; footprint Resistor_SMD:R_0201_0603Metric -> Resistor_SMD:R_1206_3216Metric
- R8: renamed from R9; footprint Resistor_SMD:R_0201_0603Metric -> Resistor_SMD:R_2010_5025Metric
- R9: renamed from R4; footprint Resistor_SMD:R_0201_0603Metric -> Resistor_SMD:R_0603_1608Metric
- renumbered C12 to C13, C19 to C15
Connections:
- net BATTERY_IN: now also C12.1
- net GND: now also C12.2, C14.2, C2.2, C3.2, E2.1, E2.3, L4.2
- net GPS_ANT: now also L3.2
- net SIM868_Vin: now also C14.1, C2.1, C3.1
- new net: E2.2, L3.1, L4.1
Other:
- moved on the sheet: C1, C15, C4, C5, C6, D5, R11
